File: pots-over-cat6.kicad_sch (KiCad schematic)
At the start: 11 parts, among them J1 615004144121, J2 615004144121, J3 615004144121, J4 615004144121, J5 615008144221

Commit message: Added PDF schematic
Other:
- company: (none) -> Evan Chodora
- title: (none) -> POTS over CAT6 Adapter
Changed lines of the file:
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@@
 	(generator_version "9.0")
 	(paper "A4")
+	(title_block
+		(title "POTS over CAT6 Adapter")
+		(date "2025-04-15")
+		(rev "1.0")
+		(company "Evan Chodora")
+	)
 	(no_connect
 		(at 118.11 114.3)
